Commit message: Update

File: urdf/physicai_arm.urdf (robot description, URDF)
Before this commit: robot physicai_arm, 8 links, 7 joints
Links:
- link base_link: geometry collision mesh filename=package://physicai_arm/urdf/assets/base_motor_holder_so101_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; collision mesh filename=package://physicai_arm/urdf/assets/base_so101_v2.stl
- link gripper_link: geometry collision mesh filename=package://physicai_arm/urdf/assets/sts3215_03a_v1.stl; collision mesh filename=package://physicai_arm/urdf/assets/wrist_roll_follower_so10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
- link lower_arm_link: geometry collision mesh filename=package://physicai_arm/urdf/assets/motor_holder_so101_wrist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; collision mesh filename=package://physicai_arm/urdf/assets/sts3215_03a_v1.stl
- link moving_jaw_so101_v1_link: geometry collision mesh filename=package://physicai_arm/urdf/assets/moving_jaw_so101_v1.stl; visual mesh filename=package://physicai_arm/urdf/assets/moving_jaw_so101_v1.stl
- link shoulder_link: geometry collision mesh filename=package://physicai_arm/urdf/assets/motor_holder_so101_base_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; collision mesh filename=package://physicai_arm/urdf/assets/rotation_pitch_so101_v1.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
- link upper_arm_link: geometry collision mesh filename=package://physicai_arm/urdf/assets/sts3215_03a_v1.stl; collision mesh filename=package://physicai_arm/urdf/assets/upper_arm_so101_v1.stl
- link wrist_link: geometry collision mesh filename=package://physicai_arm/urdf/assets/sts3215_03a_no_horn_v1.s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; collision mesh filename=package://physicai_arm/urdf/assets/wrist_roll_pitch_so101_v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
